File: audio_controller_3x2.kicad_pcb (KiCad board)
At the start: 2 copper layers, 70.5 x 41.9 mm, 24 parts, among them J1 AUDIO_JACK_3.5MM, U1 SGTL5000, U2 AP7313_1.5V, U3 LM48310

Commit message: Progress towards v1.2.
Parts:
- moved U1 5.08 mm to (135.9, 88.9)
Connections:
- J1 pad 1: (no net) -> /HP_VGND
- MDB1 pad 10: (no net) -> Net-(MDB1-Pad10)
- MDB1 pad 12: (no net) -> Net-(MDB1-Pad12)
- MDB1 pad 14: (no net) -> Net-(MDB1-Pad14)
- MDB1 pad 15: (no net) -> Net-(MDB1-Pad15)
- MDB1 pad 16: (no net) -> Net-(MDB1-Pad16)
- MDB1 pad 17: (no net) -> Net-(MDB1-Pad17)
- MDB1 pad 2: (no net) -> Net-(MDB1-Pad2)
- MDB1 pad 20: (no net) -> Net-(MDB1-Pad20)
- MDB1 pad 21: (no net) -> Net-(MDB1-Pad21)
- MDB1 pad 24: (no net) -> Net-(MDB1-Pad24)
- MDB1 pad 25: (no net) -> Net-(MDB1-Pad25)
- MDB1 pad 28: (no net) -> Net-(MDB1-Pad28)
- MDB1 pad 29: (no net) -> Net-(MDB1-Pad29)
- MDB1 pad 3: (no net) -> Net-(MDB1-Pad3)
- MDB1 pad 30: (no net) -> Net-(MDB1-Pad30)
- MDB1 pad 4: (no net) -> Net-(MDB1-Pad4)
- MDB1 pad 5: (no net) -> Net-(MDB1-Pad5)
- MDB1 pad AREF: (no net) -> Net-(MDB1-PadAREF)
- MDB1 pad VDD: (no net) -> VDD
- U1 pad 11: (no net) -> Net-(U1-Pad11)
- U1 pad 12: (no net) -> Net-(U1-Pad12)
- U1 pad 13: (no net) -> Net-(U1-Pad13)
- U1 pad 14: (no net) -> Net-(U1-Pad14)
- U1 pad 15: (no net) -> Net-(U1-Pad15)
- U1 pad 16: (no net) -> Net-(U1-Pad16)
- U1 pad 18: (no net) -> Net-(U1-Pad18)
- U1 pad 4: GND -> /HP_VGND
- U3 pad 6: Net-(U3-Pad6) -> (no net)
Routing:
- net /SDA: track 87.9 -> 47.9 mm
- net /HP_L: track 11.2 -> 33.4 mm
- net VEE: track 64.4 -> 83.3 mm, vias 0 -> 1
- net /HP_VGND: track 0.00 -> 15.9 mm
- net /LRCLK: track 39.7 -> 53.6 mm, vias 1 -> 0
- net GND: track 148.0 -> 161.8 mm, vias 3 -> 1
- net +1V5: track 25.1 -> 15.2 mm
- net Net-(C2-Pad1): track 29.0 -> 19.9 mm
- net /I2STX: track 39.8 -> 48.6 mm, vias 1 -> 0
- net /MCLK: track 32.3 -> 25.4 mm, vias 0 -> 1
- net /HP_R: track 18.4 -> 13.3 mm
- net +3V3: track 134.9 -> 139.9 mm
- net Net-(C4-Pad1): track 15.8 -> 20.1 mm
- net /I2SRX: track 30.2 -> 27.0 mm, vias 1 -> 0
- net /SCL: track 52.8 -> 55.3 mm, vias 1 -> 0
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- removed copper zone on B.Cu, net GND
- removed copper zone on F.Cu, net GND
Other:
- net class Default: trace_width 0.25 -> 0.254
- net class SUPERPOWER: trace_width 0.4064 -> 0.3556
- net class VGND added: clearance 0.1016, trace_width 0.4064, via_dia 0.889, via_drill 0.635
- board text added: "Janelia Modular Device audio_controller part_number: 1151 10/2017 ver 1.2 3x2"
- board text removed: "Janelia Modular Device audio_controller part_number: 1151 09/2017 ver 1.1 3x2"

Commit message: Finished version 1.2.
Connections:
- net /SPEAKER_ENABLE renamed /PCB_SPEAKER_ENABLE
- MDB1 pad 10: Net-(MDB1-Pad10) -> (no net)
- MDB1 pad 12: Net-(MDB1-Pad12) -> (no net)
- MDB1 pad 14: Net-(MDB1-Pad14) -> (no net)
- MDB1 pad 15: Net-(MDB1-Pad15) -> (no net)
- MDB1 pad 16: Net-(MDB1-Pad16) -> (no net)
- MDB1 pad 17: Net-(MDB1-Pad17) -> (no net)
- MDB1 pad 2: Net-(MDB1-Pad2) -> (no net)
- MDB1 pad 20: Net-(MDB1-Pad20) -> (no net)
- MDB1 pad 21: Net-(MDB1-Pad21) -> (no net)
- MDB1 pad 24: Net-(MDB1-Pad24) -> (no net)
- MDB1 pad 25: Net-(MDB1-Pad25) -> (no net)
- MDB1 pad 28: Net-(MDB1-Pad28) -> (no net)
- MDB1 pad 29: Net-(MDB1-Pad29) -> (no net)
- MDB1 pad 3: Net-(MDB1-Pad3) -> (no net)
- MDB1 pad 30: Net-(MDB1-Pad30) -> (no net)
- MDB1 pad 4: Net-(MDB1-Pad4) -> (no net)
- MDB1 pad 5: Net-(MDB1-Pad5) -> (no net)
- MDB1 pad AREF: Net-(MDB1-PadAREF) -> (no net)
- MDB1 pad VDD: VDD -> (no net)
- U1 pad 11: Net-(U1-Pad11) -> (no net)
- U1 pad 12: Net-(U1-Pad12) -> (no net)
- U1 pad 13: Net-(U1-Pad13) -> (no net)
- U1 pad 14: Net-(U1-Pad14) -> (no net)
- U1 pad 15: Net-(U1-Pad15) -> (no net)
- U1 pad 16: Net-(U1-Pad16) -> (no net)
- U1 pad 18: Net-(U1-Pad18) -> (no net)
- U3 pad 6: (no net) -> Net-(U3-Pad6)
Other:
- board text added: "PCB Speaker"
- board text added: "Stereo Speaker Output 3.5mm 1/8" Mini Plug"
- board text removed: "Stereo Output 3.5mm 1/8" Mini Plug"
