File: audio_controller_3x2.sch (KiCad schematic (older format))
At the start: 1 part

Commit message: Progress towards v1.0.
Parts:
- added C1, C3, C6: 0.1uF, audio_controller_3x2:SM1210, symbol 0.1uF
- added C2, C5, C7: 2.2uF, audio_controller_3x2:SM1210, symbol 2.2uF
- added C4: 0.15uF, audio_controller_3x2:SM1210, symbol 0.15uF
- added J1: AUDIO_JACK_3.5MM, audio_controller_3x2:AUDIO_JACK_3.5MM_3PIN, symbol AUDIO_JACK_3.5MM
- added L1: 600@100MHz, audio_controller_3x2:SM1210, symbol 600@100MHz
- added R1, R2: 2.21k, audio_controller_3x2:SM1210, symbol 2.21k
- added U1: SGTL5000, audio_controller_3x2:QFN-5x5-32, symbol SGTL5000
- added U2: AP7313_1.5V, audio_controller_3x2:SOT-23-3, symbol AP7313_1.5V
Connections:
- net labels added: +1V5, +3.3V, BCLK, HP_L, HP_R, HP_VGND, I2SRX, I2STX, LRCLK, MCLK, SCL, SDA
- wire segments 8 -> 74
- no-connect marks 29 -> 28

Commit message: Finished version 1.0.
Parts:
- U1: symbol SGTL5000 -> SGTL5000-RESCUE-audio_controller_3x2
Changed lines of the file:
@@
 EESchema Schematic File Version 2
+LIBS:audio_controller_3x2-rescue
 LIBS:power
 LIBS:device
@@
 LRCLK
 $Comp
-L SGTL5000 U1
+L SGTL5000-RESCUE-audio_controller_3x2 U1
 U 1 1 58D57661
 P 5750 4650

Commit message: Added LM48310.
Parts:
- added SP1: SPEAKER_8OHM_300MW, audio_controller_3x2:SPEAKER_8OHM_300MW, symbol SPEAKER_8OHM_300MW
Connections:
- no-connect marks 28 -> 30
Changed lines of the file:
@@
 LIBS:audio_controller_3x2
 LIBS:components
-LIBS:audio_controller_3x2-cache
 EELAYER 26 0
 EELAYER END
@@
 Title "audio_controller_3x2"
 Date ""
-Rev "1.0"
+Rev "1.1"
 Comp "Janelia"
 Comment1 ""
@@
 $EndComp
 Connection ~ 6400 3150
+$Comp
+L SPEAKER_8OHM_300MW SP1
+U 1 1 59B97E9C
+P 7500 1850
+F 0 "SP1" H 7450 1950 50  0000 C CNN
+F 1 "SPEAKER_8OHM_300MW" V 7700 1800 50  0000 C CNN
+F 2 "audio_controller_3x2:SPEAKER_8OHM_300MW" H 7500 1650 50  0001 C CNN
+F 3 "" H 7490 1800 50  0001 C CNN
+F 4 "digikey" H 7650 2175 60  0001 C CNN "Vendor"
+F 5 "102-3539-1-ND" H 7750 2275 60  0001 C CNN "PartNumber"
+F 6 "SPEAKER 8OHM 300MW TOP PORT 87DB" H 7850 2375 60  0001 C CNN "Description"
+	1    7500 1850
+	1    0    0    -1
+$EndComp
+NoConn ~ 7300 1850
+NoConn ~ 7300 1950
 $EndSCHEMATC

Commit message: Updated 0.1uF capacitors.
Parts:
- added U?: LM48310, audio_controller_3x2:10-WFDFN_EXPOSED_PAD, symbol LM48310
- C1, C3, C6: Description CAP CER 0.1UF 50V 10% X7R 1210 -> CAP CER 0.1UF 100V X7R 1210; PartNumber 478-3586-1-ND -> 399-13229-1-ND
Connections:
- net labels added: AGND, AMP+, AMP-, DAC, SPEAKER_ENABLE
- wire segments 74 -> 87
- no-connect marks 30 -> 26
Changed lines of the file:
@@
 LIBS:audio_controller_3x2
 LIBS:components
+LIBS:audio_controller_3x2-cache
 EELAYER 26 0
 EELAYER END
@@
 NoConn ~ 1400 1000
 NoConn ~ 1400 1100
-NoConn ~ 1400 1200
 NoConn ~ 1400 1300
 NoConn ~ 1400 1400
 NoConn ~ 1400 1500
-NoConn ~ 1400 1600
 NoConn ~ 1400 1700
 NoConn ~ 1400 1800
@@
 NoConn ~ 1400 2200
 NoConn ~ 3900 800
-NoConn ~ 3900 1000
 NoConn ~ 3900 1400
 NoConn ~ 3900 1500
@@
 NoConn ~ 3900 2000
 NoConn ~ 3900 2100
-NoConn ~ 3900 2300
 $Comp
 L VEE #PWR05
@@
 F 3 "" H 1900 4350 60  0000 C CNN
 F 4 "digikey" H 2000 4550 60  0001 C CNN "Vendor"
-F 5 "478-3586-1-ND" H 2100 4650 60  0001 C CNN "PartNumber"
-F 6 "CAP CER 0.1UF 50V 10% X7R 1210" H 2200 4750 60  0001 C CNN "Description"
+F 5 "399-13229-1-ND" H 2100 4650 60  0001 C CNN "PartNumber"
+F 6 "CAP CER 0.1UF 100V X7R 1210" H 2200 4750 60  0001 C CNN "Description"
 	1    1900 4350
 	1    0    0    -1
@@
 F 3 "" H 5350 3400 60  0000 C CNN
 F 4 "digikey" H 5450 3600 60  0001 C CNN "Vendor"
-F 5 "478-3586-1-ND" H 5550 3700 60  0001 C CNN "PartNumber"
-F 6 "CAP CER 0.1UF 50V 10% X7R 1210" H 5650 3800 60  0001 C CNN "Description"
+F 5 "399-13229-1-ND" H 5550 3700 60  0001 C CNN "PartNumber"
+F 6 "CAP CER 0.1UF 100V X7R 1210" H 5650 3800 60  0001 C CNN "Description"
 	1    5350 3400
 	1    0    0    -1
@@
 F 3 "" H 6400 3400 60  0000 C CNN
 F 4 "digikey" H 6500 3600 60  0001 C CNN "Vendor"
-F 5 "478-3586-1-ND" H 6600 3700 60  0001 C CNN "PartNumber"
-F 6 "CAP CER 0.1UF 50V 10% X7R 1210" H 6700 3800 60  0001 C CNN "Description"
+F 5 "399-13229-1-ND" H 6600 3700 60  0001 C CNN "PartNumber"
+F 6 "CAP CER 0.1UF 100V X7R 1210" H 6700 3800 60  0001 C CNN "Description"
 	1    6400 3400
 	1    0    0    -1
@@
 L SPEAKER_8OHM_300MW SP1
 U 1 1 59B97E9C
-P 7500 1850
-F 0 "SP1" H 7450 1950 50  0000 C CNN
-F 1 "SPEAKER_8OHM_300MW" V 7700 1800 50  0000 C CNN
-F 2 "audio_controller_3x2:SPEAKER_8OHM_300MW" H 7500 1650 50  0001 C CNN
-F 3 "" H 7490 1800 50  0001 C CNN
-F 4 "digikey" H 7650 2175 60  0001 C CNN "Vendor"
-F 5 "102-3539-1-ND" H 7750 2275 60  0001 C CNN "PartNumber"
-F 6 "SPEAKER 8OHM 300MW TOP PORT 87DB" H 7850 2375 60  0001 C CNN "Description"
-	1    7500 1850
-	1    0    0    -1
-$EndComp
-NoConn ~ 7300 1850
-NoConn ~ 7300 1950
+P 9650 1400
+F 0 "SP1" H 9600 1500 50  0000 C CNN
+F 1 "SPEAKER_8OHM_300MW" V 9850 1350 50  0000 C CNN
+F 2 "audio_controller_3x2:SPEAKER_8OHM_300MW" H 9650 1200 50  0001 C CNN
+F 3 "" H 9640 1350 50  0001 C CNN
+F 4 "digikey" H 9800 1725 60  0001 C CNN "Vendor"
+F 5 "102-3539-1-ND" H 9900 1825 60  0001 C CNN "PartNumber"
+F 6 "SPEAKER 8OHM 300MW TOP PORT 87DB" H 10000 1925 60  0001 C CNN "Description"
+	1    9650 1400
+	1    0    0    -1
+$EndComp
+$Comp
+L LM48310 U?
+U 1 1 59B9B19E
+P 8550 1350
+F 0 "U?" H 8950 1650 60  0000 C CNN
+F 1 "LM48310" H 8200 1650 60  0000 C CNN
+F 2 "audio_controller_3x2:10-WFDFN_EXPOSED_PAD" H 8850 1550 60  0001 C CNN
+F 3 "" H 8550 1350 60  0001 C CNN
+F 4 "digikey" H 9050 1750 60  0001 C CNN "Vendor"
+F 5 "LM48310SD/NOPBCT-ND" H 9150 1850 60  0001 C CNN "PartNumber"
+F 6 "IC AMP AUDIO PWR 2.6W MONO 10SON" H 9250 1950 60  0001 C CNN "Description"
+	1    8550 1350
+	1    0    0    -1
+$EndComp
+Wire Wire Line
+	9150 1400 9450 1400
+Wire Wire Line
+	9150 1500 9450 1500
+Text Label 9200 1400 0    60   ~ 0
+AMP+
+Text Label 9200 1500 0    60   ~ 0
+AMP-
+NoConn ~ 9150 1200
+$Comp
+L VEE #PWR?
+U 1 1 59B9B7F7
+P 8550 900
+F 0 "#PWR?" H 4300 50  50  0001 C CNN
+F 1 "VEE" H 8567 1073 50  0000 C CNN
+F 2 "" H 4300 200 50  0001 C CNN
+F 3 "" H 4300 200 50  0001 C CNN
+	1    8550 900
+	1    0    0    -1
+$EndComp
+Wire Wire Line
+	8500 1000 8500 950
+Wire Wire Line
+	8500 950  8600 950
+Wire Wire Line
+	8600 950  8600 1000
+Wire Wire Line
+	8550 950  8550 900
+Connection ~ 8550 950
+Wire Wire Line
+	3900 1000 4000 1000
+Wire Wire Line
+	3900 2300 4000 2300
+Text Label 4000 2300 0    60   ~ 0
+DAC
+Text Label 4000 1000 0    60   ~ 0
+AGND
+Text Label 1300 1600 2    60   ~ 0
+SPEAKER_ENABLE
+NoConn ~ 1400 1200
+Wire Wire Line
+	1300 1600 1400 1600
+$Comp
+L GND #PWR?
+U 1 1 59B99483
+P 8550 1750
+F 0 "#PWR?" H 7350 150 50  0001 C CNN
+F 1 "GND" H 8555 1577 50  0000 C CNN
+F 2 "" H 7350 400 50  0001 C CNN
+F 3 "" H 7350 400 50  0001 C CNN
+	1    8550 1750
+	1    0    0    -1
+$EndComp
+Wire Wire Line
+	8550 1700 8550 1750
+Text Label 7850 1300 2    60   ~ 0
+SPEAKER_ENABLE
+Wire Wire Line
+	7850 1300 7950 1300
+$Comp
+L VEE #PWR?
+U 1 1 59B99ACA
+P 7900 1150
+F 0 "#PWR?" H 3650 300 50  0001 C CNN
+F 1 "VEE" H 7917 1323 50  0000 C CNN
+F 2 "" H 3650 450 50  0001 C CNN
+F 3 "" H 3650 450 50  0001 C CNN
+	1    7900 1150
+	1    0    0    -1
+$EndComp
+Wire Wire Line
+	7900 1150 7900 1200
+Wire Wire Line
+	7900 1200 7950 1200
 $EndSCHEMATC

Commit message: Added speaker and amplifier.
Parts:
- removed U1: SGTL5000, audio_controller_3x2:QFN-5x5-32, symbol SGTL5000-RESCUE-audio_controller_3x2
- added C10, C11: 1uF, audio_controller_3x2:SM1210, symbol 1uF
- added C12: 2.2uF, audio_controller_3x2:SM1210, symbol 2.2uF
- added C13: 0.1uF, audio_controller_3x2:SM1210, symbol 0.1uF
- added C8, C9: 3.3nF, audio_controller_3x2:SM1210, symbol 3.3nF
- added R3, R4: 2.21k, audio_controller_3x2:SM1210, symbol 2.21k
- added U1: SGTL5000, audio_controller_3x2:QFN-5x5-32, symbol SGTL5000
- gave numbers to parts that had none: 1
Connections:
- wire segments 87 -> 112
Changed lines of the file:
@@
 Text Label 4000 1200 0    60   ~ 0
 LRCLK
-$Comp
-L SGTL5000-RESCUE-audio_controller_3x2 U1
-U 1 1 58D57661
-P 5750 4650
-F 0 "U1" H 6300 5350 60  0000 C CNN
-F 1 "SGTL5000" H 6200 3800 60  0000 C CNN
-F 2 "audio_controller_3x2:QFN-5x5-32" H 6050 5250 60  0001 C CNN
-F 3 "" H 5750 4650 60  0001 C CNN
-F 4 "digikey" H 6250 5450 60  0001 C CNN "Vendor"
-F 5 "SGTL5000XNAA3R2CT-ND" H 6350 5550 60  0001 C CNN "PartNumber"
-F 6 "Stereo Audio Interface 32-QFN" H 6450 5650 60  0001 C CNN "Description"
-	1    5750 4650
-	1    0    0    -1
-$EndComp
 Text Label 4850 4100 2    60   ~ 0
 SDA
@@
 $EndComp
 $Comp
-L LM48310 U?
+L LM48310 U3
 U 1 1 59B9B19E
 P 8550 1350
-F 0 "U?" H 8950 1650 60  0000 C CNN
+F 0 "U3" H 8950 1650 60  0000 C CNN
 F 1 "LM48310" H 8200 1650 60  0000 C CNN
 F 2 "audio_controller_3x2:10-WFDFN_EXPOSED_PAD" H 8850 1550 60  0001 C CNN
@@
 NoConn ~ 9150 1200
 $Comp
-L VEE #PWR?
+L VEE #PWR04
 U 1 1 59B9B7F7
 P 8550 900
-F 0 "#PWR?" H 4300 50  50  0001 C CNN
+F 0 "#PWR04" H 4300 50  50  0001 C CNN
 F 1 "VEE" H 8567 1073 50  0000 C CNN
 F 2 "" H 4300 200 50  0001 C CNN
@@
 	1300 1600 1400 1600
 $Comp
-L GND #PWR?
+L GND #PWR06
 U 1 1 59B99483
 P 8550 1750
-F 0 "#PWR?" H 7350 150 50  0001 C CNN
+F 0 "#PWR06" H 7350 150 50  0001 C CNN
 F 1 "GND" H 8555 1577 50  0000 C CNN
 F 2 "" H 7350 400 50  0001 C CNN
@@
 	7850 1300 7950 1300
 $Comp
-L VEE #PWR?
+L VEE #PWR02
 U 1 1 59B99ACA
 P 7900 1150
-F 0 "#PWR?" H 3650 300 50  0001 C CNN
+F 0 "#PWR02" H 3650 300 50  0001 C CNN
 F 1 "VEE" H 7917 1323 50  0000 C CNN
 F 2 "" H 3650 450 50  0001 C CNN
@@
 Wire Wire Line
 	7900 1200 7950 1200
+$Comp
+L 1uF C10
+U 1 1 59B9A980
+P 7600 1450
+F 0 "C10" V 7650 1400 40  0000 R CNN
+F 1 "1uF" H 7600 1450 30  0000 C CNN
+F 2 "audio_controller_3x2:SM1210" H 7638 1300 30  0001 C CNN
+F 3 "" H 7600 1450 60  0000 C CNN
+F 4 "digikey" H 7700 1650 60  0001 C CNN "Vendor"
+F 5 "399-8219-1-ND" H 7800 1750 60  0001 C CNN "PartNumber"
+F 6 "CAP CER 1UF 100V X7R 1210" H 7900 1850 60  0001 C CNN "Description"
+	1    7600 1450
+	0    -1   -1   0
+$EndComp
+$Comp
+L 1uF C11
+U 1 1 59B9AEDB
+P 7600 1650
+F 0 "C11" V 7650 1600 40  0000 R CNN
+F 1 "1uF" H 7600 1650 30  0000 C CNN
+F 2 "audio_controller_3x2:SM1210" H 7638 1500 30  0001 C CNN
+F 3 "" H 7600 1650 60  0000 C CNN
+F 4 "digikey" H 7700 1850 60  0001 C CNN "Vendor"
+F 5 "399-8219-1-ND" H 7800 1950 60  0001 C CNN "PartNumber"
+F 6 "CAP CER 1UF 100V X7R 1210" H 7900 2050 60  0001 C CNN "Description"
+	1    7600 1650
+	0    -1   -1   0
+$EndComp
+Wire Wire Line
+	7950 1500 7900 1500
+Wire Wire Line
+	7900 1500 7900 1650
+Wire Wire Line
+	7900 1650 7800 1650
+Wire Wire Line
+	7950 1400 7850 1400
+Wire Wire Line
+	7850 1400 7850 1450
+Wire Wire Line
+	7850 1450 7800 1450
+$Comp
+L 2.21k R3
+U 1 1 59B9B27D
+P 6800 1450
+F 0 "R3" V 6700 1450 40  0000 C CNN
+F 1 "2.21k" V 6800 1450 40  0000 C CNN
+F 2 "audio_controller_3x2:SM1210" V 6730 1450 30  0001 C CNN
+F 3 "" H 6800 1450 30  0000 C CNN
+F 4 "digikey" V 6980 1550 60  0001 C CNN "Vendor"
+F 5 "P2.21KAACT-ND" V 7080 1650 60  0001 C CNN "PartNumber"
+F 6 "RES SMD 2.21K OHM 1% 1/2W 1210" V 7180 1750 60  0001 C CNN "Description"
+	1    6800 1450
+	0    1    1    0
+$EndComp
+$Comp
+L 2.21k R4
+U 1 1 59B9B412
+P 6800 1650
+F 0 "R4" V 6700 1650 40  0000 C CNN
+F 1 "2.21k" V 6800 1650 40  0000 C CNN
+F 2 "audio_controller_3x2:SM1210" V 6730 1650 30  0001 C CNN
+F 3 "" H 6800 1650 30  0000 C CNN
+F 4 "digikey" V 6980 1750 60  0001 C CNN "Vendor"
+F 5 "P2.21KAACT-ND" V 7080 1850 60  0001 C CNN "PartNumber"
+F 6 "RES SMD 2.21K OHM 1% 1/2W 1210" V 7180 1950 60  0001 C CNN "Description"
+	1    6800 1650
+	0    1    1    0
+$EndComp
+Wire Wire Line
+	7050 1450 7400 1450
+Wire Wire Line
+	7050 1650 7400 1650
+Wire Wire Line
+	6550 1450 6450 1450
+Wire Wire Line
+	6550 1650 6450 1650
+Text Label 6450 1450 2    60   ~ 0
+DAC
+Text Label 6450 1650 2    60   ~ 0
+AGND
+$Comp
+L 3.3nF C9
+U 1 1 59B9D598
+P 7350 2000
+F 0 "C9" H 7350 2100 40  0000 L CNN
+F 1 "3.3nF" H 7350 2000 30  0000 C CNN
+F 2 "audio_controller_3x2:SM1210" H 7388 1850 30  0001 C CNN
+F 3 "" H 7350 2000 60  0000 C CNN
+F 4 "digikey" H 7450 2200 60  0001 C CNN "Vendor"
+F 5 "478-5964-1-ND" H 7550 2300 60  0001 C CNN "PartNumber"
+F 6 "CAP CER 3300PF 2KV X7R 1210" H 7650 2400 60  0001 C CNN "Description"
+	1    7350 2000
+	1    0    0    -1
+$EndComp
+$Comp
+L 3.3nF C8
+U 1 1 59B9D911
+P 7150 2000
+F 0 "C8" H 7150 2100 40  0000 L CNN
+F 1 "3.3nF" H 7150 2000 30  0000 C CNN
+F 2 "audio_controller_3x2:SM1210" H 7188 1850 30  0001 C CNN
+F 3 "" H 7150 2000 60  0000 C CNN
+F 4 "digikey" H 7250 2200 60  0001 C CNN "Vendor"
+F 5 "478-5964-1-ND" H 7350 2300 60  0001 C CNN "PartNumber"
+F 6 "CAP CER 3300PF 2KV X7R 1210" H 7450 2400 60  0001 C CNN "Description"
+	1    7150 2000
+	1    0    0    -1
+$EndComp
+Wire Wire Line
+	7150 1800 7150 1450
+Connection ~ 7150 1450
+Wire Wire Line
+	7350 1800 7350 1650
+Connection ~ 7350 1650
+Wire Wire Line
+	7150 2200 7150 2250
+Wire Wire Line
+	7150 2250 7350 2250
+Wire Wire Line
+	7350 2250 7350 2200
+Wire Wire Line
+	7250 2250 7250 2350
+Wire Wire Line
+	7250 2350 7300 2350
+Connection ~ 7250 2250
+Text Label 7300 2350 0    60   ~ 0
+AGND
+$Comp
+L 2.2uF C12
+U 1 1 59B9E31B
+P 8900 2300
+F 0 "C12" H 8900 2400 40  0000 L CNN
+F 1 "2.2uF" H 8900 2300 30  0000 C CNN
+F 2 "audio_controller_3x2:SM1210" H 8938 2150 30  0001 C CNN
+F 3 "" H 8900 2300 60  0000 C CNN
+F 4 "digikey" H 9000 2500 60  0001 C CNN "Vendor"
+F 5 "478-3591-1-ND" H 9100 2600 60  0001 C CNN "PartNumber"
+F 6 "2.2uF 50V Ceramic Capacitor X7R 1210" H 9200 2700 60  0001 C CNN "Description"
+	1    8900 2300
+	1    0    0    -1
+$EndComp
+$Comp
+L 0.1uF C13
+U 1 1 59B9E451
+P 9100 2300
+F 0 "C13" H 9100 2400 40  0000 L CNN
+F 1 "0.1uF" H 9100 2300 30  0000 C CNN
+F 2 "audio_controller_3x2:SM1210" H 9138 2150 30  0001 C CNN
+F 3 "" H 9100 2300 60  0000 C CNN
+F 4 "digikey" H 9200 2500 60  0001 C CNN "Vendor"
+F 5 "399-13229-1-ND" H 9300 2600 60  0001 C CNN "PartNumber"
+F 6 "CAP CER 0.1UF 100V X7R 1210" H 9400 2700 60  0001 C CNN "Description"
+	1    9100 2300
+	1    0    0    -1
+$EndComp
+$Comp
+L VEE #PWR015
+U 1 1 59B9E60A
+P 9000 2000
+F 0 "#PWR015" H 4750 1150 50  0001 C CNN
+F 1 "VEE" H 9017 2173 50  0000 C CNN
+F 2 "" H 4750 1300 50  0001 C CNN
+F 3 "" H 4750 1300 50  0001 C CNN
+	1    9000 2000
+	1    0    0    -1
+$EndComp
+$Comp
+L GND #PWR025
+U 1 1 59B9E675
+P 9000 2600
+F 0 "#PWR025" H 7800 1000 50  0001 C CNN
+F 1 "GND" H 9005 2427 50  0000 C CNN
+F 2 "" H 7800 1250 50  0001 C CNN
+F 3 "" H 7800 1250 50  0001 C CNN
+	1    9000 2600
+	1    0    0    -1
+$EndComp
+Wire Wire Line
+	8900 2100 8900 2050
+Wire Wire Line
+	8900 2050 9100 2050
+Wire Wire Line
+	9100 2050 9100 2100
+Wire Wire Line
+	8900 2500 8900 2550
+Wire Wire Line
+	8900 2550 9100 2550
+Wire Wire Line
+	9100 2550 9100 2500
+Wire Wire Line
+	9000 2550 9000 2600
+Connection ~ 9000 2550
+Wire Wire Line
+	9000 2000 9000 2050
+Connection ~ 9000 2050
+$Comp
+L SGTL5000 U1
+U 1 1 59B9F587
+P 5750 4650
+F 0 "U1" H 6250 5350 60  0000 C CNN
+F 1 "SGTL5000" H 5350 5350 60  0000 C CNN
+F 2 "audio_controller_3x2:QFN-5x5-32" H 6050 5250 60  0001 C CNN
+F 3 "" H 5750 4650 60  0001 C CNN
+F 4 "digikey" H 6250 5450 60  0001 C CNN "Vendor"
+F 5 "SGTL5000XNAA3R2CT-ND" H 6350 5550 60  0001 C CNN "PartNumber"
+F 6 "Stereo Audio Interface 32-QFN" H 6450 5650 60  0001 C CNN "Description"
+	1    5750 4650
+	1    0    0    -1
+$EndComp
 $EndSCHEMATC

Commit message: Fixed 0.15uF part number.
Parts:
- C4: PartNumber 399-11615-1-ND -> 399-15599-1-ND
Changed lines of the file:
@@
 F 3 "" H 4700 5150 60  0000 C CNN
 F 4 "digikey" H 4800 5350 60  0001 C CNN "Vendor"
-F 5 "399-11615-1-ND" H 4900 5450 60  0001 C CNN "PartNumber"
+F 5 "399-15599-1-ND" H 4900 5450 60  0001 C CNN "PartNumber"
 F 6 "0.15uF 100V Ceramic Capacitor X7R 1210" H 5000 5550 60  0001 C CNN "Description"
 	1    4700 5150

Commit message: Progress towards v1.2.
Changed lines of the file:
@@
-EESchema Schematic File Version 2
-LIBS:audio_controller_3x2-rescue
+EESchema Schematic File Version 3
 LIBS:power
-LIBS:device
-LIBS:transistors
-LIBS:conn
-LIBS:linear
-LIBS:regul
-LIBS:74xx
-LIBS:cmos4000
-LIBS:adc-dac
-LIBS:memory
-LIBS:xilinx
-LIBS:microcontrollers
-LIBS:dsp
-LIBS:microchip
-LIBS:analog_switches
-LIBS:motorola
-LIBS:texas
-LIBS:intel
-LIBS:audio
-LIBS:interface
-LIBS:digital-audio
-LIBS:philips
-LIBS:display
-LIBS:cypress
-LIBS:siliconi
-LIBS:opto
-LIBS:atmel
-LIBS:contrib
-LIBS:valves
 LIBS:audio_controller_3x2
 LIBS:components
@@
 Title "audio_controller_3x2"
 Date ""
-Rev "1.1"
+Rev "1.2"
 Comp "Janelia"
 Comment1 ""
@@
 Connection ~ 5650 5700
 Wire Wire Line
-	5750 5650 5750 5750
+	5750 5700 5750 5750
 Connection ~ 5750 5700
 Wire Wire Line
