File: audio_controller_3x2.sch (KiCad schematic (older format))
At the start: 24 parts, among them J1 AUDIO_JACK_3.5MM, U1 SGTL5000, U2 AP7313_1.5V, U3 LM48310

Commit message: Finished version 1.2.
Connections:
- net labels added: PCB_SPEAKER_ENABLE
- net labels removed: SPEAKER_ENABLE
Changed lines of the file:
@@
 L MODULAR_DEVICE_BASE_3X2_MALE MDB1
 U 1 1 589B6745
-P 2650 1550
-F 0 "MDB1" H 2650 2547 60  0000 C CNN
-F 1 "MODULAR_DEVICE_BASE_3X2_MALE" H 2650 2441 60  0000 C CNN
-F 2 "audio_controller_3x2:MODULAR_DEVICE_BASE_3X2_MALE" H 600 1050 60  0001 C CNN
-F 3 "" H 650 2750 60  0000 C CNN
-F 4 "digikey" H 600 1150 60  0001 C CNN "Vendor"
-F 5 "S1011E-16-ND" H 600 1250 60  0001 C CNN "PartNumber"
-F 6 "16 Position Header Through Hole Male Pins" H 600 1350 60  0001 C CNN "Description"
-F 7 "2" H 1900 1250 60  0001 C CNN "PartCount"
-	1    2650 1550
+P 2900 1650
+F 0 "MDB1" H 2900 2647 60  0000 C CNN
+F 1 "MODULAR_DEVICE_BASE_3X2_MALE" H 2900 2541 60  0000 C CNN
+F 2 "audio_controller_3x2:MODULAR_DEVICE_BASE_3X2_MALE" H 850 1150 60  0001 C CNN
+F 3 "" H 900 2850 60  0000 C CNN
+F 4 "digikey" H 850 1250 60  0001 C CNN "Vendor"
+F 5 "S1011E-16-ND" H 850 1350 60  0001 C CNN "PartNumber"
+F 6 "16 Position Header Through Hole Male Pins" H 850 1450 60  0001 C CNN "Description"
+F 7 "2" H 2150 1350 60  0001 C CNN "PartCount"
+	1    2900 1650
 	1    0    0    -1
 $EndComp
@@
 L VDD #PWR01
 U 1 1 589B67C3
-P 1350 750
-F 0 "#PWR01" H 100 -400 50  0001 C CNN
-F 1 "VDD" H 1367 923 50  0000 C CNN
-F 2 "" H 100 -250 50  0001 C CNN
-F 3 "" H 100 -250 50  0001 C CNN
-	1    1350 750
+P 1600 850
+F 0 "#PWR01" H 350 -300 50  0001 C CNN
+F 1 "VDD" H 1617 1023 50  0000 C CNN
+F 2 "" H 350 -150 50  0001 C CNN
+F 3 "" H 350 -150 50  0001 C CNN
+	1    1600 850
 	1    0    0    -1
 $EndComp
@@
 L PWR_FLAG #FLG02
 U 1 1 589B67D9
-P 1100 750
-F 0 "#FLG02" H -150 -175 50  0001 C CNN
-F 1 "PWR_FLAG" H 1100 924 50  0000 C CNN
-F 2 "" H -150 -250 50  0001 C CNN
-F 3 "" H -150 -250 50  0001 C CNN
-	1    1100 750
+P 1350 850
+F 0 "#FLG02" H 100 -75 50  0001 C CNN
+F 1 "PWR_FLAG" H 1350 1024 50  0000 C CNN
+F 2 "" H 100 -150 50  0001 C CNN
+F 3 "" H 100 -150 50  0001 C CNN
+	1    1350 850
 	1    0    0    -1
 $EndComp
@@
 L GND #PWR03
 U 1 1 589B67FE
-P 700 950
-F 0 "#PWR03" H -500 -650 50  0001 C CNN
-F 1 "GND" H 705 777 50  0000 C CNN
-F 2 "" H -500 -400 50  0001 C CNN
-F 3 "" H -500 -400 50  0001 C CNN
-	1    700  950
+P 950 1050
+F 0 "#PWR03" H -250 -550 50  0001 C CNN
+F 1 "GND" H 955 877 50  0000 C CNN
+F 2 "" H -250 -300 50  0001 C CNN
+F 3 "" H -250 -300 50  0001 C CNN
+	1    950  1050
 	1    0    0    -1
 $EndComp
@@
 L PWR_FLAG #FLG04
 U 1 1 589B6835
-P 700 750
-F 0 "#FLG04" H -550 -175 50  0001 C CNN
-F 1 "PWR_FLAG" H 700 924 50  0000 C CNN
-F 2 "" H -550 -250 50  0001 C CNN
-F 3 "" H -550 -250 50  0001 C CNN
-	1    700  750
-	1    0    0    -1
-$EndComp
-NoConn ~ 1400 1000
-NoConn ~ 1400 1100
-NoConn ~ 1400 1300
-NoConn ~ 1400 1400
-NoConn ~ 1400 1500
-NoConn ~ 1400 1700
-NoConn ~ 1400 1800
-NoConn ~ 1400 2000
-NoConn ~ 1400 2200
-NoConn ~ 3900 800
-NoConn ~ 3900 1400
-NoConn ~ 3900 1500
-NoConn ~ 3900 1800
-NoConn ~ 3900 1900
-NoConn ~ 3900 2000
-NoConn ~ 3900 2100
+P 950 850
+F 0 "#FLG04" H -300 -75 50  0001 C CNN
+F 1 "PWR_FLAG" H 950 1024 50  0000 C CNN
+F 2 "" H -300 -150 50  0001 C CNN
+F 3 "" H -300 -150 50  0001 C CNN
+	1    950  850
+	1    0    0    -1
+$EndComp
+NoConn ~ 1650 1100
+NoConn ~ 1650 1200
+NoConn ~ 1650 1400
+NoConn ~ 1650 1500
+NoConn ~ 1650 1600
+NoConn ~ 1650 1800
+NoConn ~ 1650 1900
+NoConn ~ 1650 2100
+NoConn ~ 1650 2300
+NoConn ~ 4150 900
+NoConn ~ 4150 1500
+NoConn ~ 4150 1600
+NoConn ~ 4150 1900
+NoConn ~ 4150 2000
+NoConn ~ 4150 2100
+NoConn ~ 4150 2200
 $Comp
 L VEE #PWR05
 U 1 1 589B69B5
-P 4450 800
-F 0 "#PWR05" H 200 -50 50  0001 C CNN
-F 1 "VEE" H 4467 973 50  0000 C CNN
-F 2 "" H 200 100 50  0001 C CNN
-F 3 "" H 200 100 50  0001 C CNN
-	1    4450 800
+P 4700 900
+F 0 "#PWR05" H 450 50  50  0001 C CNN
+F 1 "VEE" H 4717 1073 50  0000 C CNN
+F 2 "" H 450 200 50  0001 C CNN
+F 3 "" H 450 200 50  0001 C CNN
+	1    4700 900
 	1    0    0    -1
 $EndComp
@@
 L PWR_FLAG #FLG06
 U 1 1 589B69CA
-P 4750 800
-F 0 "#FLG06" H 3500 -125 50  0001 C CNN
-F 1 "PWR_FLAG" H 4750 974 50  0000 C CNN
-F 2 "" H 3500 -200 50  0001 C CNN
-F 3 "" H 3500 -200 50  0001 C CNN
-	1    4750 800
-	1    0    0    -1
-$EndComp
-Text Label 1300 1900 2    60   ~ 0
+P 5000 900
+F 0 "#FLG06" H 3750 -25 50  0001 C CNN
+F 1 "PWR_FLAG" H 5000 1074 50  0000 C CNN
+F 2 "" H 3750 -100 50  0001 C CNN
+F 3 "" H 3750 -100 50  0001 C CNN
+	1    5000 900
+	1    0    0    -1
+$EndComp
+Text Label 1550 2000 2    60   ~ 0
 BCLK
-Text Label 4000 2200 0    60   ~ 0
+Text Label 4250 2300 0    60   ~ 0
 I2SRX
-Text Label 4000 1700 0    60   ~ 0
+Text Label 4250 1800 0    60   ~ 0
 SDA
-Text Label 4000 1600 0    60   ~ 0
+Text Label 4250 1700 0    60   ~ 0
 SCL
-Text Label 4000 1300 0    60   ~ 0
+Text Label 4250 1400 0    60   ~ 0
 I2STX
-Text Label 4000 1200 0    60   ~ 0
+Text Label 4250 1300 0    60   ~ 0
 LRCLK
 Text Label 4850 4100 2    60   ~ 0
@@
 L +3.3V #PWR014
 U 1 1 58D58DDB
-P 5000 950
-F 0 "#PWR014" H 5000 800 50  0001 C CNN
-F 1 "+3.3V" H 5015 1123 50  0000 C CNN
-F 2 "" H 5000 950 50  0001 C CNN
-F 3 "" H 5000 950 50  0001 C CNN
-	1    5000 950
+P 5250 1050
+F 0 "#PWR014" H 5250 900 50  0001 C CNN
+F 1 "+3.3V" H 5265 1223 50  0000 C CNN
+F 2 "" H 5250 1050 50  0001 C CNN
+F 3 "" H 5250 1050 50  0001 C CNN
+	1    5250 1050
 	1    0    0    -1
 $EndComp
@@
 L PWR_FLAG #FLG015
 U 1 1 58D58EBA
-P 5300 1050
-F 0 "#FLG015" H 4050 125 50  0001 C CNN
-F 1 "PWR_FLAG" H 5300 1224 50  0000 C CNN
-F 2 "" H 4050 50  50  0001 C CNN
-F 3 "" H 4050 50  50  0001 C CNN
-	1    5300 1050
+P 5550 1150
+F 0 "#FLG015" H 4300 225 50  0001 C CNN
+F 1 "PWR_FLAG" H 5550 1324 50  0000 C CNN
+F 2 "" H 4300 150 50  0001 C CNN
+F 3 "" H 4300 150 50  0001 C CNN
+	1    5550 1150
 	1    0    0    -1
 $EndComp
@@
 Text Label 4400 3750 0    60   ~ 0
 SCL
-Text Label 1300 2100 2    60   ~ 0
+Text Label 1550 2200 2    60   ~ 0
 MCLK
 Wire Wire Line
-	1100 750  1100 800
-Wire Wire Line
-	1100 800  1400 800
-Wire Wire Line
-	1350 750  1350 800
-Connection ~ 1350 800
-Wire Wire Line
-	700  750  700  950
-Wire Wire Line
-	700  900  1400 900
-Connection ~ 700  900
-Wire Wire Line
-	4750 900  4750 800
-Wire Wire Line
-	3900 900  4750 900
-Wire Wire Line
-	4450 800  4450 900
-Connection ~ 4450 900
-Wire Wire Line
-	1400 1900 1300 1900
-Wire Wire Line
-	3900 2200 4000 2200
-Wire Wire Line
-	3900 1700 4000 1700
-Wire Wire Line
-	3900 1600 4000 1600
-Wire Wire Line
-	3900 1300 4000 1300
-Wire Wire Line
-	3900 1200 4000 1200
+	1350 850  1350 900
+Wire Wire Line
+	1350 900  1650 900
+Wire Wire Line
+	1600 850  1600 900
+Connection ~ 1600 900
+Wire Wire Line
+	950  850  950  1050
+Wire Wire Line
+	950  1000 1650 1000
+Connection ~ 950  1000
+Wire Wire Line
+	5000 1000 5000 900
+Wire Wire Line
+	4150 1000 5000 1000
+Wire Wire Line
+	4700 900  4700 1000
+Connection ~ 4700 1000
+Wire Wire Line
+	1650 2000 1550 2000
+Wire Wire Line
+	4150 2300 4250 2300
+Wire Wire Line
+	4150 1800 4250 1800
+Wire Wire Line
+	4150 1700 4250 1700
+Wire Wire Line
+	4150 1400 4250 1400
+Wire Wire Line
+	4150 1300 4250 1300
 Wire Wire Line
 	4950 4100 4850 4100
@@
 	2700 4550 2700 4600
 Wire Wire Line
-	3900 1100 5300 1100
-Wire Wire Line
-	5000 1100 5000 950
-Wire Wire Line
-	5300 1100 5300 1050
-Connection ~ 5000 1100
+	4150 1200 5550 1200
+Wire Wire Line
+	5250 1200 5250 1050
+Wire Wire Line
+	5550 1200 5550 1150
+Connection ~ 5250 1200
 Connection ~ 2700 4100
 Wire Wire Line
@@
 	4350 3100 4350 3050
 Wire Wire Line
-	1400 2100 1300 2100
+	1650 2200 1550 2200
 Connection ~ 1700 4100
 Connection ~ 1900 4100
-NoConn ~ 1400 2300
+NoConn ~ 1650 2400
 $Comp
 L PWR_FLAG #FLG025
@@
 Connection ~ 8550 950
 Wire Wire Line
-	3900 1000 4000 1000
-Wire Wire Line
-	3900 2300 4000 2300
-Text Label 4000 2300 0    60   ~ 0
+	4150 1100 4250 1100
+Wire Wire Line
+	4150 2400 4250 2400
+Text Label 4250 2400 0    60   ~ 0
 DAC
-Text Label 4000 1000 0    60   ~ 0
+Text Label 4250 1100 0    60   ~ 0
 AGND
-Text Label 1300 1600 2    60   ~ 0
-SPEAKER_ENABLE
-NoConn ~ 1400 1200
-Wire Wire Line
-	1300 1600 1400 1600
+Text Label 1550 1700 2    60   ~ 0
+PCB_SPEAKER_ENABLE
+NoConn ~ 1650 1300
+Wire Wire Line
+	1550 1700 1650 1700
 $Comp
 L GND #PWR06
@@
 	8550 1700 8550 1750
 Text Label 7850 1300 2    60   ~ 0
-SPEAKER_ENABLE
+PCB_SPEAKER_ENABLE
 Wire Wire Line
 	7850 1300 7950 1300
