File: audio_controller_3x2.sch (KiCad schematic (older format))
At the start: 24 parts, among them J1 AUDIO_JACK_3.5MM, U1 SGTL5000, U2 AP7313_1.5V, U3 LM48310

Commit message: Updated to v4.
Parts:
- C1, C13, C3, C6: symbol 0.1uF -> audio_controller_3x2:0.1uF
- C10, C11: symbol 1uF -> audio_controller_3x2:1uF
- C12, C2, C5, C7: symbol 2.2uF -> audio_controller_3x2:2.2uF
- C4: symbol 0.15uF -> audio_controller_3x2:0.15uF
- C8, C9: symbol 3.3nF -> audio_controller_3x2:3.3nF
- J1: symbol AUDIO_JACK_3.5MM -> audio_controller_3x2:AUDIO_JACK_3.5MM
- L1: symbol 600@100MHz -> audio_controller_3x2:600@100MHz
- MDB1: symbol MODULAR_DEVICE_BASE_3X2_MALE -> audio_controller_3x2:MODULAR_DEVICE_BASE_3X2_MALE
- R1, R2, R3, R4: symbol 2.21k -> audio_controller_3x2:2.21k
- SP1: symbol SPEAKER_8OHM_300MW -> audio_controller_3x2:SPEAKER_8OHM_300MW
- U1: symbol SGTL5000 -> audio_controller_3x2:SGTL5000
- U2: symbol AP7313_1.5V -> audio_controller_3x2:AP7313_1.5V
- U3: symbol LM48310 -> audio_controller_3x2:LM48310
Connections:
- wire segments 112 -> 134
